File: PCB/FLL.kicad_pcb (KiCad board)
At the start: 2 copper layers, 11 parts, among them U1 LM317L_SOT-89, U2 MCP73831-2-MC

Commit message: chore: Update PCB design configuration and remove unnecessary files
Parts:
- removed C2: 0,47uF, Capacitor_SMD:C_Elec_6.3x5.4
- removed D1: LED Blau, LED_THT:LED_D3.0mm_Horizontal_O6.35mm_Z10.0mm
- removed POT4: 240Ω, Resistor_SMD:R_0603_1608Metric_Pad0.98x0.95mm_HandSolder
- removed U2: MCP73831-2-MC, Package_DFN_QFN:DFN-8-1EP_3x2mm_P0.5mm_EP1.7x1.4mm
- added C4: 4,5uF, Capacitor_THT:CP_Axial_L10.0mm_D4.5mm_P15.00mm_Horizontal, F.Cu at (145.9, 37.3)
- added U3: LM317L_SOT-89, Package_TO_SOT_SMD:SOT-89-3, F.Cu at (170.5, 47.5)
- C1: value 4,5uF -> 1uF
- C3: value 1uF -> 0,47uF
- POT2: value 1kΩ -> 1,4kΩ
- POT3: value 1,4kΩ -> 1kΩ
- U1: value LM317L_SOT-89 -> MCP73831-2-MC; footprint Package_TO_SOT_SMD:SOT-89-3 -> Package_DFN_QFN:DFN-8-1EP_3x2mm_P0.5mm_EP1.7x1.4mm
- moved POT3 43.9 mm to (175.6, 36.5), turned to -90 degrees
- moved C1 40.8 mm to (146.0, 42.5)
- moved POT2 34.5 mm to (164.5, 44.5)
- moved POT1 33.8 mm to (165.5, 48.1), turned to 90 degrees
- moved U1 31.3 mm to (169.1, 39.4)
- moved C3 30.5 mm to (146.0, 47.7)
- moved F1 22.2 mm to (176.4, 49.5), turned to 90 degrees
Connections:
- C1 pad 1: +7.5V -> +16V
- C1 pad 2: -16V -> /7,3V |1A Output
- C3 pad 2: /7,3V |1A Output -> +16V
- POT1 pad 1: Net-(D1|2,2V1-K) -> Net-(U3-VO)
- POT1 pad 2: +16V -> Net-(U3-ADJ)
- POT2 pad 1: Net-(U1-PROG) -> +16V
- POT2 pad 2: -16V -> Net-(U3-ADJ)
- POT3 pad 1: +16V -> Net-(U1-PROG)
- POT3 pad 2: Net-(U3-ADJ) -> -16V
- U1 pad 1: Net-(U3-ADJ) -> /7,3V |1A Output
- U1 pad 2: Net-(U3-VO) -> /7,3V |1A Output
- U1 pad 3: +16V -> +7.5V
Routing:
- net /7,3V |1A Output: track 94.2 -> 30.1 mm
- net +7.5V: track 25.2 -> 49.0 mm
- net -16V: track 38.6 -> 21.9 mm, vias 1 -> 2
- net Net-(U3-VO): track 28.8 -> 12.6 mm
- net Net-(U1-PROG): track 13.2 -> 29.2 mm
- net Net-(U3-ADJ): track 20.1 -> 10.0 mm
- net +16V: track 46.0 -> 39.5 mm
- net Net-(D1|2,2V1-K): track 6.09 -> 0.00 mm
- net +1V0: track 0.00 -> 5.02 mm, vias 0 -> 1
- net (no net): vias 2 -> 0
Other:
- board text added: "${REFERENCE}"

Commit message: chore: Update PCB design configuration and remove unnecessary files
Connections:
- net /7,3V |1A Output renamed Net-(C1-Pad2)
- C1 pad 1: +16V -> GND
- C3 pad 1: +16V -> GND
- POT2 pad 1: +16V -> GND
Routing:
- net GND: track 0.00 -> 30.9 mm, vias 0 -> 1
- net +16V: track 39.5 -> 11.5 mm
- net Net-(C1-Pad2): track 30.1 -> 31.8 mm
- net Net-(U1-PROG): track 29.2 -> 30.4 mm
- net +7.5V: track 49.0 -> 50.1 mm, vias 0 -> 1
- net -16V: track 21.9 -> 22.4 mm
