File: PCB/FLL.kicad_pcb (KiCad board)
At the start: 2 copper layers, 18.4 x 23.5 mm, 16 parts, among them U2 MCP73831-2-OT, U3 LM317L_SOT-89

Commit message: chore: Update plot directory for KiCad project
Parts:
- moved POT1 1.52 mm to (30.0, 19.0)
- moved ? 1.45 mm to (19.4, 29.5)
- moved ? 1.45 mm to (16.9, 29.5)
- moved C3 0.95 mm to (17.9, 25.5)
- moved F1 0.60 mm to (29.6, 25.0)
Routing:
- net Net-(U3-VO): track 14.3 -> 16.4 mm
- net Net-(U3-ADJ): track 11.5 -> 13.2 mm
- net GND: track 13.8 -> 15.2 mm
Changed lines of the file:
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@@
 		(pcbplotparams
 			(layerselection 0x00010fc_ffffffff)
-			(plot_on_all_layers_selection 0x0000000_00000000)
+			(plot_on_all_layers_selection 0x00010fc_80000001)
 			(disableapertmacros no)
 			(usegerberextensions no)
@@
 			(sketchpadsonfab no)
 			(subtractmaskfromsilk no)
-			(outputformat 1)
+			(outputformat 4)
 			(mirror no)
 			(drillshape 0)
 			(scaleselection 1)
-			(outputdirectory "")
+			(outputdirectory "../Material/")
 		)
 	)
@@
 	(footprint "C0805C474K5RACTU:C0805"
 		(layer "F.Cu")
-		(at 17.9125 24.55)
+		(at 17.889669 25.5)
 		(descr "C0805")
 		(tags "Capacitor")
@@
 	(footprint ""
 		(layer "F.Cu")
-		(at 19.4125 28.05)
+		(at 19.4125 29.5)
 		(property "Reference" ""
 			(at 0 0 0)
@@
 	(footprint "Fuse:Fuse_Bourns_MF-RG300"
 		(layer "F.Cu")
-		(at 29 25 -90)
+		(at 29.6 25 -90)
 		(descr "PTC Resettable Fuse, Ihold = 3.0A, Itrip=5.1A, http://www.bourns.com/docs/Product-Datasheets/mfrg.pdf")
 		(tags "ptc resettable fuse polyfuse THT")
@@
 	(footprint "1206L075THYR:1206L05015YR"
 		(layer "F.Cu")
-		(at 28.9 20.05 90)
+		(at 30 19 90)
 		(descr "1206L035")
 		(tags "Resettable Fuse")
@@
 	(footprint ""
 		(layer "F.Cu")
-		(at 16.9125 28.05)
+		(at 16.9125 29.5)
 		(property "Reference" ""
 			(at 0 0 0)
@@
 	)
 	(gr_text "GND"
-		(at 17.9125 30.05 0)
+		(at 20.5 27.5 0)
 		(layer "F.SilkS")
 		(effects
@@
 	)
 	(segment
-		(start 22.5375 21.05)
-		(end 22.625 20.9625)
+		(start 30 20.475)
+		(end 23.1125 20.475)
 		(width 0.2)
 		(layer "F.Cu")
@@
 	)
 	(segment
-		(start 28.9 20.9625)
-		(end 28.9 24.9)
+		(start 23.1125 20.475)
+		(end 22.5375 21.05)
+		(width 0.2)
+		(layer "F.Cu")
+		(net 2)
+	)
+	(segment
+		(start 30 20.475)
+		(end 30 24.6)
 		(width 0.2)
 		(layer "F.Cu")
@@
 	)
 	(segment
-		(start 22.625 20.9625)
-		(end 28.9 20.9625)
+		(start 30 24.6)
+		(end 29.6 25)
 		(width 0.2)
 		(layer "F.Cu")
@@
 	)
 	(segment
-		(start 23.4 19.55)
-		(end 23.8125 19.1375)
-		(width 0.2)
-		(layer "F.Cu")
-		(net 3)
-	)
-	(segment
 		(start 22.45 19.55)
-		(end 23.4 19.55)
+		(end 27.975 19.55)
 		(width 0.2)
 		(layer "F.Cu")
@@
 	)
 	(segment
-		(start 23.8125 19.1375)
-		(end 28.9 19.1375)
-		(width 0.2)
-		(layer "F.Cu")
-		(net 3)
-	)
-	(segment
 		(start 20.45 17.55)
 		(end 22.45 19.55)
@@
 	)
 	(segment
+		(start 27.975 19.55)
+		(end 30 17.525)
+		(width 0.2)
+		(layer "F.Cu")
+		(net 3)
+	)
+	(segment
 		(start 24.3125 35.55)
 		(end 24.95 36.1875)
@@
 	)
 	(segment
+		(start 16.9125 25.577169)
+		(end 16.989669 25.5)
+		(width 0.2)
+		(layer "F.Cu")
+		(net 5)
+	)
+	(segment
 		(start 17.4005 20.662)
 		(end 17.0125 21.05)
@@
 	)
 	(segment
-		(start 16.9125 28.05)
-		(end 19.4125 28.05)
+		(start 16.9125 29.5)
+		(end 19.4125 29.5)
 		(width 0.2)
 		(layer "F.Cu")
@@
 	)
 	(segment
-		(start 17.0125 24.55)
-		(end 17.0125 25.45)
+		(start 16.995869 25.4938)
+		(end 16.989669 25.5)
 		(width 0.2)
 		(layer "F.Cu")
@@
 	)
 	(segment
-		(start 17.0125 21.983262)
-		(end 17.0125 24.55)
+		(start 16.9125 29.5)
+		(end 16.9125 25.577169)
+		(width 0.2)
+		(layer "F.Cu")
+		(net 5)
+	)
+	(segment
+		(start 16.995869 21.234208)
+		(end 16.995869 25.4938)
 		(width 0.2)
 		(layer "F.Cu")
@@
 	)
 	(segment
-		(start 16.995869 21.234208)
-		(end 16.995869 21.966631)
-		(width 0.2)
-		(layer "F.Cu")
-		(net 5)
-	)
-	(segment
-		(start 16.9125 25.55)
-		(end 16.9125 28.05)
-		(width 0.2)
-		(layer "F.Cu")
-		(net 5)
-	)
-	(segment
-		(start 17.0125 25.45)
-		(end 16.9125 25.55)
-		(width 0.2)
-		(layer "F.Cu")
-		(net 5)
-	)
-	(segment
-		(start 16.995869 21.966631)
-		(end 17.0125 21.983262)
-		(width 0.2)
-		(layer "F.Cu")
-		(net 5)
+		(start 21.95 25.5)
+		(end 22.4 25.05)
+		(width 0.2)
+		(layer "F.Cu")
+		(net 6)
 	)
 	(segment
@@
 	)
 	(segment
-		(start 22.4 25.05)
-		(end 19.3125 25.05)
-		(width 0.2)
-		(layer "F.Cu")
-		(net 6)
-	)
-	(segment
-		(start 19.3125 25.05)
-		(end 18.8125 24.55)
+		(start 18.789669 25.5)
+		(end 21.95 25.5)
 		(width 0.2)
 		(layer "F.Cu")
@@
 	(segment
 		(start 26.85 33.9125)
-		(end 26.85 31.05)
+		(end 26.85 31.65)
 		(width 0.2)
 		(layer "F.Cu")
@@
 	)
 	(segment
-		(start 26.85 31.05)
-		(end 27.8 30.1)
-		(width 0.2)
-		(layer "F.Cu")
+		(start 26.85 31.65)
+		(end 28.4 30.1)
+		(width 0.2)
+		(layer "F.Cu")

Commit message: Rework ALL
Parts:
- POT1: value 1206L05015YR -> 240Ω; footprint 1206L075THYR:1206L05015YR -> ERJ-2RHD1401X:ERJ2RKD1004X
- moved POT1 1.80 mm to (29.0, 20.5), turned to 180 degrees
- renumbered C4 to C1
Connections:
- C3 pad 2: Net-(U3-VI) -> Net-(M1|12V/1A1-+)
- POT1 pad 1: Net-(U3-VO) -> (no net)
- POT1 pad 2: Net-(U3-ADJ) -> (no net)
- U2 pad 1: +1V0 -> unconnected-(U2-STAT-Pad1)
- U3 pad 3: Net-(U3-VI) -> Net-(M1|12V/1A1-+)
Routing:
- net Net-(U3-VO): track 16.4 -> 4.26 mm
- net Net-(U3-ADJ): track 13.2 -> 4.85 mm
Other:
- board size 18.4 x 23.5 mm -> 19 x 23.5 mm
